File: EAGLE/PedestrianController.sch (EAGLE design)
At the start: 0 parts

Commit message: Finished schematics.
Parts:
- added CON1: FTDI, PedestrianController:MA04-1
- added CON2: DS3231, PedestrianController:MA06-1
- added CON3: AC110V, PedestrianController:MKDSN1,5/2-5,08
- added CON4: SIGNAL, PedestrianController:MKDSN1,5/3-5,08
- added IC1: ESP-WROOM-02, PedestrianController:ESP-WROOM-02FRONT-FACE
- added PROGSW, RSTSW: (no value), PedestrianController:10-XX
- added R1, R2, R3, R4, R5, R6, R7: 10K, PedestrianController:R-US_0204/7
- added SSR1, SSR2: S101T02, PedestrianController:S101T02
Connections:
- new net +3V3: CON1.1, CON2.2, IC1.3V3, R3.2, R4.2, R5.2, R6.2
- new net AC110V: CON3-1.KL, SSR1.DS2, SSR2.DS2
- new net ACCOM: CON3-2.KL, CON4-3.KL
- new net GND: CON1.2, CON2.1, IC1.GND1, IC1.GND2, IC1.GND3, PROGSW.P, PROGSW.P1, R1.1, R2.1, R7.1, RSTSW.P, RSTSW.P1
- new net N$1: IC1.IO0, PROGSW.S, PROGSW.S1, R4.1
- new net N$10: IC1.RST, R3.1, RSTSW.S, RSTSW.S1
- new net N$13: IC1.EN, R5.1
- new net N$14: IC1.IO2, R6.1
- new net N$15: IC1.IO15, R7.2
- new net N$2: IC1.IO13, SSR2.A
- new net N$3: R2.2, SSR1.K
- new net N$4: R1.2, SSR2.K
- new net N$9: IC1.IO12, SSR1.A
- new net RXD: CON1.4, IC1.RXD
- new net SCL: CON2.4, IC1.IO5
- new net SDA: CON2.3, IC1.IO4
- new net STOP: CON4-2.KL, SSR2.DS1
- new net TXD: CON1.3, IC1.TXD
- new net WALK: CON4-1.KL, SSR1.DS1
