File: EAGLE/PedestrianController.brd (EAGLE design)
At the start: 57.8 x 85 mm, 28 parts, among them CON1 FTDI, CON2 DS3231, CON3 AC110V, CON4 SIGNAL, IC1 ESP-WROOM-02, SW1 RSTSW, SW2 PROGSW

Commit message: Adjust resistor values by GPIO current specs.
Parts:
- LED1, LED2, LED3: value (none) -> RH156
- R1, R2: value 100 -> 200
Changed lines of the file:
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@@
 <attribute name="OC_NEWARK" value="36M3542" x="8.715" y="77.7" size="1.778" layer="27" display="off"/>
 </element>
-<element name="R1" library="PedestrianController" package="0204/7" package3d_urn="urn:adsk.eagle:package:25945/1" value="100" x="30.74" y="49" rot="R270"/>
-<element name="R2" library="PedestrianController" package="0204/7" package3d_urn="urn:adsk.eagle:package:25945/1" value="100" x="27.74" y="49" rot="R270"/>
+<element name="R1" library="PedestrianController" package="0204/7" package3d_urn="urn:adsk.eagle:package:25945/1" value="200" x="30.74" y="49" rot="R270"/>
+<element name="R2" library="PedestrianController" package="0204/7" package3d_urn="urn:adsk.eagle:package:25945/1" value="200" x="27.74" y="49" rot="R270"/>
 <element name="R3" library="PedestrianController" package="0204/7" package3d_urn="urn:adsk.eagle:package:25945/1" value="10K" x="43.74" y="68"/>
 <element name="R4" library="PedestrianController" package="0204/7" package3d_urn="urn:adsk.eagle:package:25945/1" value="10K" x="43.74" y="76.8"/>
@@
 <element name="R8" library="PedestrianController" package="0204/7" package3d_urn="urn:adsk.eagle:package:25945/1" value="510" x="22" y="49" rot="R270"/>
 <element name="R9" library="PedestrianController" package="0204/7" package3d_urn="urn:adsk.eagle:package:25945/1" value="510" x="25" y="49" rot="R270"/>
-<element name="LED1" library="PedestrianController" package="LED3MM" package3d_urn="urn:adsk.eagle:package:15797/1" value="" x="6" y="43">
+<element name="LED1" library="PedestrianController" package="LED3MM" package3d_urn="urn:adsk.eagle:package:15797/1" value="RH156" x="6" y="43">
 <attribute name="MF" value="VISHAY SEMICONDUCTOR" x="6" y="43" size="1.778" layer="27" display="off"/>
 <attribute name="OC_FARNELL" value="1612437" x="6" y="43" size="1.778" layer="27" display="off"/>
 </element>
-<element name="LED2" library="PedestrianController" package="LED3MM" package3d_urn="urn:adsk.eagle:package:15797/1" value="" x="14" y="43">
+<element name="LED2" library="PedestrianController" package="LED3MM" package3d_urn="urn:adsk.eagle:package:15797/1" value="RH156" x="14" y="43">
 <attribute name="MF" value="VISHAY SEMICONDUCTOR" x="14" y="43" size="1.778" layer="27" display="off"/>
 <attribute name="OC_FARNELL" value="1612437" x="14" y="43" size="1.778" layer="27" display="off"/>
 </element>
-<element name="R10" library="PedestrianController" package="0204/7" package3d_urn="urn:adsk.eagle:package:25945/1" value="510" x="30.74" y="57" rot="R180"/>
-<element name="LED3" library="PedestrianController" package="LED3MM" package3d_urn="urn:adsk.eagle:package:15797/1" value="" x="23" y="57">
+<element name="R10" library="PedestrianController" package="0204/7" package3d_urn="urn:adsk.eagle:package:25945/1" value="510" x="30.74" y="57" rot="R180">
+<attribute name="SPICEPREFIX" value="R" x="30.74" y="57" size="1.778" layer="27" rot="R180" display="off"/>
+</element>
+<element name="LED3" library="PedestrianController" package="LED3MM" package3d_urn="urn:adsk.eagle:package:15797/1" value="RH156" x="23" y="57">
 <attribute name="MF" value="VISHAY SEMICONDUCTOR" x="23" y="57" size="1.778" layer="27" display="off"/>
 <attribute name="OC_FARNELL" value="1612437" x="23" y="57" size="1.778" layer="27" display="off"/>
